Commit message: irp6_defs : added missing joint.

File: irp6_robot/irp6_defs/robots/irp6p.urdf.xacro (robot description, xacro)
@@ -45,5 +45,5 @@
       <origin rpy="0 0 0.0" xyz="0 0 0.2"/>
       <geometry>
-        <box size="0.2 0.25 0.4"/>
+        <box size="0.22 0.25 0.4"/>
       </geometry>
     </visual>
@@ -51,10 +51,10 @@
       <origin rpy="0 0 0.0" xyz="0 0 0.2"/>
       <geometry>
-        <box size="0.2 0.25 0.4"/>
+        <box size="0.22 0.25 0.4"/>
       </geometry>
     </collision>
   </link>
   <joint name="joint2" type="revolute">
-    <origin rpy="1.57 0 0" xyz="0.0 0.0 0.4"/>
+    <origin rpy="-1.57 0 0" xyz="0.0 0.0 0.4"/>
     <axis xyz="0 0 1"/>
     <limit lower="-1.57" upper="1.57" effort="10.0" velocity="10.0" />
@@ -69,18 +69,18 @@
     </inertial>
     <visual>
-      <origin rpy="0 0 0.0" xyz="0 0.2 0.0"/>
+      <origin rpy="0 0 0.0" xyz="0.2 0.0 0.0"/>
       <geometry>
-        <box size="0.15 0.4 0.2"/>
+        <box size="0.4 0.10 0.2"/>
       </geometry>
     </visual>
     <collision>
-      <origin rpy="0 0 0.0" xyz="0 0.2 0.0"/>
+      <origin rpy="0 0 0.0" xyz="0.2 0.0 0.0"/>
       <geometry>
-        <box size="0.15 0.4 0.2"/>
+        <box size="0.4 0.10 0.2"/>
       </geometry>
     </collision>
   </link>
   <joint name="joint3" type="revolute">
-    <origin rpy="0 0 -1.57" xyz="0.0 0.45 0.0"/>
+    <origin rpy="0 0 0.0" xyz="0.45 0.0 0.0"/>
     <axis xyz="0 0 1"/>
     <limit lower="-1.57" upper="1.57" effort="10.0" velocity="10.0" />
@@ -97,5 +97,5 @@
       <origin rpy="0 0 0.0" xyz="0 0.30 0.0"/>
       <geometry>
-        <box size="0.15 0.67 0.2"/>
+        <box size="0.10 0.67 0.15"/>
       </geometry>
     </visual>
@@ -103,5 +103,5 @@
       <origin rpy="0 0 0.0" xyz="0 0.3 0.0"/>
       <geometry>
-        <box size="0.15 0.67 0.2"/>
+        <box size="0.10 0.67 0.15"/>
       </geometry>
     </collision>
@@ -109,5 +109,5 @@
   <joint name="joint4" type="revolute">
     <origin rpy="0 0 0" xyz="0.0 0.67 0.0"/>
-    <axis xyz="1 0 0"/>
+    <axis xyz="0 0 1"/>
     <limit lower="-1.57" upper="1.57" effort="10.0" velocity="10.0" />
     <parent link="link3"/>
@@ -122,6 +122,6 @@
   </link>
   <joint name="joint5" type="revolute">
-    <origin rpy="0 0 0" xyz="0.0 0.0 0.0"/>
-    <axis xyz="0 1 0"/>
+    <origin rpy="-1.57 0 0" xyz="0.0 0.0 0.0"/>
+    <axis xyz="0 0 1"/>
     <limit lower="0.0" upper="3.14" effort="10.0" velocity="10.0" />
     <parent link="link4"/>
@@ -134,4 +134,30 @@
       <inertia ixx="0.1" ixy="0" ixz="0" iyy="0.1" iyz="0" izz="0.1"/>
     </inertial>
+    <visual>
+      <origin rpy="0 0 0.0" xyz="0 0.0 0.1"/>
+      <geometry>
+        <cylinder radius="0.025" length="0.2"/>
+      </geometry>
+    </visual>
+  </link>
+  <joint name="joint6" type="revolute">
+    <origin rpy="1.57 0 0" xyz="0.0 0.0 0.2"/>
+    <axis xyz="0 0 1"/>
+    <limit lower="0.0" upper="3.14" effort="10.0" velocity="10.0" />
+    <parent link="link5"/>
+    <child link="link6"/>
+  </joint>
+  <link name="link6">
+    <inertial>
+      <mass value="0.1"/>
+      <origin xyz="0.0 0.0 0.0"/>
+      <inertia ixx="0.1" ixy="0" ixz="0" iyy="0.1" iyz="0" izz="0.1"/>
+    </inertial>
+    <visual>
+      <origin rpy="0 0 0.0" xyz="0 0.0 0.0"/>
+      <geometry>
+        <cylinder radius="0.05" length="0.3"/>
+      </geometry>
+    </visual>
   </link>
 </robot>

Commit message: irp6_defs : meshes added. irp6_defs : joints limits aplied.

File: irp6_robot/irp6_defs/robots/irp6p.urdf.xacro (robot description, xacro)
@@ -5,4 +5,5 @@
        xmlns:xacro="http://ros.org/wiki/fixme"
        xmlns:interface="http://playerstage.sourceforge.net/gazebo/xmlschema/#interface">
+  <property name="M_PI" value="3.14159"/>
   <link name="base_link">
     <inertial>
@@ -13,13 +14,4 @@
                izz="1.0" />
     </inertial>
-    <visual>
-      <origin xyz="0.0 0 0.15" rpy="0 0 0" />
-      <geometry>
-        <box size="0.40 0.4 0.3" />
-      </geometry>
-      <material name="Cyan">
-        <color rgba="0.5 0.5 0.5 1.0"/>
-      </material>
-    </visual>
     <collision>
       <origin xyz="0 0 0.15" rpy="0 0 0" />
@@ -32,5 +24,5 @@
     <origin rpy="0 0 0" xyz="0.0 0.0 0.3"/>
     <axis xyz="0 0 1"/>
-    <limit lower="-3.0" upper="3.0" effort="10.0" velocity="10.0" />
+    <limit lower="-2.96705973" upper="2.96705973" effort="10.0" velocity="10.0" />
     <parent link="base_link"/>
     <child link="link1"/>
@@ -43,7 +35,7 @@
     </inertial>
     <visual>
-      <origin rpy="0 0 0.0" xyz="0 0 0.2"/>
+      <origin rpy="-1.57 0 0.0" xyz="0 0 0.4"/>
       <geometry>
-        <box size="0.22 0.25 0.4"/>
+        <mesh filename="package://irp6_defs/meshes/link1.3ds" scale="0.01 0.01 0.01" />
       </geometry>
     </visual>
@@ -56,7 +48,7 @@
   </link>
   <joint name="joint2" type="revolute">
-    <origin rpy="-1.57 0 0" xyz="0.0 0.0 0.4"/>
+    <origin rpy="${-0.5 * M_PI} 0 0" xyz="0.0 0.0 0.4"/>
     <axis xyz="0 0 1"/>
-    <limit lower="-1.57" upper="1.57" effort="10.0" velocity="10.0" />
+    <limit lower="-2.26892803" upper="-0.872664626" effort="10.0" velocity="10.0" />
     <parent link="link1"/>
     <child link="link2"/>
@@ -69,7 +61,7 @@
     </inertial>
     <visual>
-      <origin rpy="0 0 0.0" xyz="0.2 0.0 0.0"/>
+      <origin rpy="0 0 0.0" xyz="0.45 0.0 0.0"/>
       <geometry>
-        <box size="0.4 0.10 0.2"/>
+        <mesh filename="package://irp6_defs/meshes/link2.3ds" scale="0.01 0.01 0.01" />
       </geometry>
     </visual>
@@ -84,5 +76,5 @@
     <origin rpy="0 0 0.0" xyz="0.45 0.0 0.0"/>
     <axis xyz="0 0 1"/>
-    <limit lower="-1.57" upper="1.57" effort="10.0" velocity="10.0" />
+    <limit lower="-0.698131701" upper="0.698131701" effort="10.0" velocity="10.0" />
     <parent link="link2"/>
     <child link="link3"/>
@@ -95,7 +87,7 @@
     </inertial>
     <visual>
-      <origin rpy="0 0 0.0" xyz="0 0.30 0.0"/>
+      <origin rpy="0 0 1.57" xyz="0 0.67 0.0"/>
       <geometry>
-        <box size="0.10 0.67 0.15"/>
+        <mesh filename="package://irp6_defs/meshes/link3.3ds" scale="0.01 0.01 0.01" />
       </geometry>
     </visual>
@@ -120,7 +112,13 @@
       <inertia ixx="0.1" ixy="0" ixz="0" iyy="0.1" iyz="0" izz="0.1"/>
     </inertial>
+    <visual>
+      <origin rpy="1.57 0 1.57" xyz="0.0 0.175 0.0"/>
+      <geometry>
+        <mesh filename="package://irp6_defs/meshes/link4.3ds" scale="0.01 0.01 0.01" />
+      </geometry>
+    </visual>
   </link>
   <joint name="joint5" type="revolute">
-    <origin rpy="-1.57 0 0" xyz="0.0 0.0 0.0"/>
+    <origin rpy="${-0.5 * M_PI} 0 0" xyz="0.0 0.0 0.0"/>
     <axis xyz="0 0 1"/>
     <limit lower="0.0" upper="3.14" effort="10.0" velocity="10.0" />
@@ -135,12 +133,12 @@
     </inertial>
     <visual>
-      <origin rpy="0 0 0.0" xyz="0 0.0 0.1"/>
+      <origin rpy="1.57 0 0.0" xyz="0.0 0.0 0.2"/>
       <geometry>
-        <cylinder radius="0.025" length="0.2"/>
+        <mesh filename="package://irp6_defs/meshes/link5.3ds" scale="0.01 0.01 0.01" />
       </geometry>
     </visual>
   </link>
   <joint name="joint6" type="revolute">
-    <origin rpy="1.57 0 0" xyz="0.0 0.0 0.2"/>
+    <origin rpy="${0.5 * M_PI} 0 0" xyz="0.0 -0.1 0.2"/>
     <axis xyz="0 0 1"/>
     <limit lower="0.0" upper="3.14" effort="10.0" velocity="10.0" />
@@ -157,5 +155,5 @@
       <origin rpy="0 0 0.0" xyz="0 0.0 0.0"/>
       <geometry>
-        <cylinder radius="0.05" length="0.3"/>
+         <mesh filename="package://irp6_defs/meshes/link6.3ds" scale="0.01 0.01 0.01" />
       </geometry>
     </visual>

Commit message: irp6_defs : collision added. irp6_launch : run_fakeservo added.

File: irp6_robot/irp6_defs/robots/irp6p.urdf.xacro (robot description, xacro)
@@ -138,4 +138,10 @@
       </geometry>
     </visual>
+    <collision>
+      <origin rpy="1.57 0 0.0" xyz="0 0.12 0.2"/>
+      <geometry>
+        <cylinder radius="0.05" length="0.30" />
+      </geometry>
+    </collision>
   </link>
   <joint name="joint6" type="revolute">
@@ -158,4 +164,26 @@
       </geometry>
     </visual>
+    <collision>
+      <origin rpy="0.0 0 0.0" xyz="0 0.0 -0.04"/>
+      <geometry>
+        <cylinder radius="0.1" length="0.08" />
+      </geometry>
+    </collision>
   </link>
+<!--
+  <joint name="laser_tilt" type="revolute">
+    <origin rpy="${0.5 * M_PI} 0 0" xyz="0.0 -0.1 2.2"/>
+    <axis xyz="0 0 1"/>
+    <limit lower="0.0" upper="3.14" effort="10.0" velocity="10.0" />
+    <parent link="base_link"/>
+    <child link="laser_link"/>
+  </joint>
+  <link name="laser_link">
+    <inertial>
+      <mass value="0.1"/>
+      <origin xyz="0.0 0.0 0.0"/>
+      <inertia ixx="0.1" ixy="0" ixz="0" iyy="0.1" iyz="0" izz="0.1"/>
+    </inertial>
+  </link>
+-->
 </robot>
